File: Modem-Hardware/Nabu_Modem.kicad_pcb (KiCad board)
At the start: 2 copper layers, 63.5 x 69.6 mm, 39 parts, among them J1 USB_C_Receptacle, J2 Nabu PC, J3 SD-Card, J4 Prog, SW1 Signal, SW2 Reset, U1 ESP-12E, U2 UA9637, U3 UA9638CD, U5 AP1117-33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

Commit message: Updated for KiCAD 7
Other:
- net class Default removed
